File: kicad/FreqCounter3203.kicad_sch (KiCad schematic)
At the start: 22 parts, among them J1 max4466_Mic_Module, J2 WCH-LINKE, SW1 OK, SW2 ↓, SW3 ↑, SW7 SWITCH_INV, U1 SEEED_GROVE, U2 OLED_0.96in_SPI, U3 CH32V003F4P6, Y1 24M

Commit message: change kicad files
Parts:
- added C5: 10u, Capacitor_SMD:C_0603_1608Metric, symbol Device:C
- added C6: 1u, Capacitor_SMD:C_0603_1608Metric, symbol Device:C
- added J3: Conn_01x07_Socket, Connector_PinSocket_2.54mm:PinSocket_1x07_P2.54mm_Vertical, symbol Connector:Conn_01x07_Socket
- added R5, R6: 5.1k, Resistor_SMD:R_0603_1608Metric, symbol FreqCounter3203-rescue:R
- added R7: 1.5k, Resistor_SMD:R_0603_1608Metric, symbol FreqCounter3203-rescue:R
- added R8, R9: 47, Resistor_SMD:R_0603_1608Metric, symbol FreqCounter3203-rescue:R
- added U4: XC6206PxxxMR, Package_TO_SOT_SMD:SOT-23-3, symbol Regulator_Linear:XC6206PxxxMR
- added U5: USB-C_16PIN, library:USB_Type_C_16Pin_Female, symbol nanbuwks:USB-C_16PIN
Connections:
- net +3V3: now also C6.2, J3.2 (Pin_2), R7.1, U4.2 (VO)
- net GND: now also C5.1, C6.1, J3.1 (Pin_1), R5.2, R6.2, U4.1 (GND), U5.A1 (GND), U5.A12 (GND), U5.B1 (GND), U5.B12 (GND)
- net at U2.3 (D0), U3.15 (PC5/SCK/T1ETR/T2CH1ETR_/SCL_/UCK/T1CH3_): now also J3.3 (Pin_3)
- net at U2.4 (D1): now also U3.16 (PC6/MOSI/T1CH1CH3N_/UCTS_/SDA_), J3.4 (Pin_4); no longer U3.14 (PC4/A2/T1CH4/MCO/T1CH1Ch2N_)
- net at U2.5 (RST), U3.17 (PC7/MISO/T1CH2_/T2CH2_/URTS_): now also J3.5 (Pin_5)
- net at U2.6 (DC): now also U3.14 (PC4/A2/T1CH4/MCO/T1CH1Ch2N_), J3.6 (Pin_6); no longer U3.16 (PC6/MOSI/T1CH1CH3N_/UCTS_/SDA_)
- net at U2.7 (CS), U3.13 (PC3/T1CH3/T1CH1N_/UCTS): now also J3.7 (Pin_7)
- net at C3.2, U3.6 (PA2/OSCO/A0/T1CH2N/OPP0/AETR2_), Y1.1: now also R9.2
- net at C2.2, U3.5 (PA1/OSCI/A1/T1CH2/OPN0), Y1.2: now also R8.2
- new net: R5.1, U5.A5 (CC1)
- new net: R7.2, R9.1, U5.A7 (DN1), U5.B7 (DN2)
- new net: R8.1, U5.A6 (DP1), U5.B6 (DP2)
- new net: R6.1, U5.B5 (CC2)
- new net +5V: C5.2, U4.3 (VI), U5.A4 (VBUS), U5.A9 (VBUS), U5.B4 (VBUS), U5.B9 (VBUS)
- no-connect marks 1 -> 3
Other:
- moved on the sheet: D1, R1
